Commit message: Fixes  - fix pathes in launch files  - add rviz  - fix configs  - fix model direction

File: urdf/camera.xacro (robot description, xacro)
@@ -1,5 +1,5 @@
 <?xml version="1.0"?>
 <robot xmlns:xacro="http://www.ros.org/wiki/xacro">
-  <xacro:macro name="my_camera" params="xyz rpy">
+  <xacro:macro name="my_camera">
     <material name="yellow">
       <color rgba="1 1 0 1"/>
@@ -22,10 +22,4 @@
       </inertial>
     </link>
-    <joint name="camera_joint" type="fixed">
-      <axis xyz="0 0 0" />
-      <origin xyz="${xyz}" rpy="${rpy}"/>
-      <parent link="base_link"/>
-      <child link="camera_link"/>
-    </joint>
     <gazebo reference="camera_link">
         <material>Gazebo/Yellow</material>

File: urdf/hexapod.xacro (robot description, xacro)
@@ -8,7 +8,13 @@
         <parent link="base_link"/>
         <child link="body"/>
-        <origin rpy="0 0 0" xyz="0 0 0"/>
+        <origin rpy="0 0 ${pi/2}" xyz="0 0 0"/>
     </joint>
-    <xacro:my_camera xyz="0 -0.1 0" rpy="0 0 ${3*pi/2}"/>
+    <xacro:my_camera/>
+    <joint name="camera_joint" type="fixed">
+      <axis xyz="0 0 0" />
+      <origin xyz="0.1 0 0" rpy="0 0 0"/>
+      <parent link="base_link"/>
+      <child link="camera_link"/>
+    </joint>
     <m_link_mesh name="body"
                 origin_rpy="0 0 0" origin_xyz="0 0 0"
