Commit message: Fix some robot params

File: urdf/hexapod.xacro (robot description, xacro)
@@ -30,8 +30,8 @@
                 type="revolute"
                 axis_xyz="0 0 1"
-                origin_rpy="0 0 0" origin_xyz="-0.040 -0.066 -0.0112"
+                origin_rpy="0 0 0" origin_xyz="-${body_legs_dx} -${body_legs_f_dy} ${body_legs_dz}"
                 parent="body" child="${link_01_name}" />
     <m_link_mesh name="${link_01_name}"
-                origin_rpy="3.14 0 0" origin_xyz="-0.033 -0.007 0"
+                origin_rpy="${pi} 0 0" origin_xyz="-${coxa_dx} -${coxa_dy} -${coxa_dz}"
                 mass="0.024357719"
                 ixx="0.0051411124" ixy="-0.00057530255" ixz="-0.000024729049"
@@ -44,8 +44,8 @@
                 type="revolute"
                 axis_xyz="0 1 0"
-                origin_rpy="0 0 3.14" origin_xyz="-0.025 0.0123 0.011"
+                origin_rpy="0 0 ${pi}" origin_xyz="-${coxa_dx - coxa_thigh_dx} ${coxa_dy - coxa_thigh_dy} -${coxa_dz - coxa_thigh_dz}"
                 parent="${link_01_name}" child="${link_02_name}" />
     <m_link_mesh name="${link_02_name}"
-                origin_rpy="1.57 0 0" origin_xyz="0.020 -0.002 -0.007"
+                origin_rpy="${pi/2} 0 0" origin_xyz="${thigh_dx} -${thigh_dz - coxa_thigh_dy} -${thigh_dy}"
                 mass="0.024357719"
                 ixx="0.0051411124" ixy="-0.00057530255" ixz="-0.000024729049"
@@ -58,8 +58,8 @@
                 type="revolute"
                 axis_xyz="0 1 0"
-                origin_rpy="0 0 0" origin_xyz="0.040 0 0"
+                origin_rpy="0 0 0" origin_xyz="${thigh_dx * 2} -${thigh_dz - tibia_dz - 0.001} 0"
                 parent="${link_02_name}" child="${link_03_name}" />
     <m_link_mesh name="${link_03_name}"
-                origin_rpy="4.712 0 3.14" origin_xyz="-0.008 0.0197 0.023"
+                origin_rpy="${3*pi/2} 0 ${pi}" origin_xyz="-${tibia_dx} ${thigh_dz - tibia_dz} ${tibia_dy}"
                 mass="0.024357719"
                 ixx="0.0051411124" ixy="-0.00057530255" ixz="-0.000024729049"
@@ -73,8 +73,8 @@
                 type="revolute"
                 axis_xyz="0 0 1"
-                origin_rpy="0 0 0" origin_xyz="0.040 -0.066 -0.0112"
+                origin_rpy="0 0 0" origin_xyz="${body_legs_dx} -${body_legs_f_dy} -${coxa_dz - body_legs_dz}"
                 parent="${link_00_name}" child="${link_04_name}" />
     <m_link_mesh name="${link_04_name}"
-                origin_rpy="3.14 0 0" origin_xyz="0.033 -0.007 0"
+                origin_rpy="${pi} 0 0" origin_xyz="${coxa_dx} -${coxa_dy} 0"
                 mass="0.024357719"
                 ixx="0.0051411124" ixy="-0.00057530255" ixz="-0.000024729049"
@@ -87,8 +87,8 @@
                 type="revolute"
                 axis_xyz="0 1 0"
-                origin_rpy="0 0 0" origin_xyz="0.025 0.0123 0.011"
+                origin_rpy="0 0 0" origin_xyz="0.025 ${coxa_thigh_dy} ${coxa_thigh_dz}"
                 parent="${link_04_name}" child="${link_05_name}" />
     <m_link_mesh name="${link_05_name}"
-                origin_rpy="1.57 0 3.14" origin_xyz="0.020 0.002 -0.007"
+                origin_rpy="${pi/2} 0 ${pi}" origin_xyz="${thigh_dx} 0.002 -${thigh_dy}"
                 mass="0.024357719"
                 ixx="0.0051411124" ixy="-0.00057530255" ixz="-0.000024729049"
@@ -104,5 +104,5 @@
                 parent="${link_05_name}" child="${link_06_name}" />
     <m_link_mesh name="${link_06_name}"
-                origin_rpy="4.712 0 0" origin_xyz="-0.008 -0.0197 0.023"
+                origin_rpy="${3*pi/2} 0 0" origin_xyz="-${tibia_dx} -${thigh_dz - tibia_dz} ${tibia_dy}"
                 mass="0.024357719"
                 ixx="0.0051411124" ixy="-0.00057530255" ixz="-0.000024729049"
@@ -116,8 +116,8 @@
                 type="revolute"
                 axis_xyz="0 0 1"
-                origin_rpy="0 0 0" origin_xyz="-0.040 0.006 -0.0112"
+                origin_rpy="0 0 0" origin_xyz="-${body_legs_dx} ${body_legs_m_dy} -${coxa_dz - body_legs_dz}"
                 parent="${link_00_name}" child="${link_07_name}" />
     <m_link_mesh name="${link_07_name}"
-                origin_rpy="3.14 0 0" origin_xyz="-0.033 -0.007 0"
+                origin_rpy="${pi} 0 0" origin_xyz="-${coxa_dx} -${coxa_dy} 0"
                 mass="0.024357719"
                 ixx="0.0051411124" ixy="-0.00057530255" ixz="-0.000024729049"
@@ -130,8 +130,8 @@
                 type="revolute"
                 axis_xyz="0 1 0"
-                origin_rpy="0 0 3.14" origin_xyz="-0.025 0.0123 0.011"
+                origin_rpy="0 0 ${pi}" origin_xyz="-0.025 ${coxa_thigh_dy} ${coxa_thigh_dz}"
                 parent="${link_07_name}" child="${link_08_name}" />
     <m_link_mesh name="${link_08_name}"
-                origin_rpy="1.57 0 0" origin_xyz="0.020 -0.002 -0.007"
+                origin_rpy="${pi/2} 0 0" origin_xyz="${thigh_dx} -0.002 -${thigh_dy}"
                 mass="0.024357719"
                 ixx="0.0051411124" ixy="-0.00057530255" ixz="-0.000024729049"
@@ -147,5 +147,5 @@
                 parent="${link_08_name}" child="${link_09_name}" />
     <m_link_mesh name="${link_09_name}"
-                origin_rpy="4.712 0 3.14" origin_xyz="-0.008 0.0197 0.023"
+                origin_rpy="${3*pi/2} 0 ${pi}" origin_xyz="-${tibia_dx} ${thigh_dz - tibia_dz} ${tibia_dy}"
                 mass="0.024357719"
                 ixx="0.0051411124" ixy="-0.00057530255" ixz="-0.000024729049"
@@ -159,8 +159,8 @@
                 type="revolute"
                 axis_xyz="0 0 1"
-                origin_rpy="0 0 0" origin_xyz="0.040 0.006 -0.0112"
+                origin_rpy="0 0 0" origin_xyz="${body_legs_dx} ${body_legs_m_dy} -${coxa_dz - body_legs_dz}"
                 parent="${link_00_name}" child="${link_10_name}" />
     <m_link_mesh name="${link_10_name}"
-                origin_rpy="3.14 0 0" origin_xyz="0.033 -0.007 0"
+                origin_rpy="${pi} 0 0" origin_xyz="${coxa_dx} -${coxa_dy} 0"
                 mass="0.024357719"
                 ixx="0.0051411124" ixy="-0.00057530255" ixz="-0.000024729049"
@@ -173,8 +173,8 @@
                 type="revolute"
                 axis_xyz="0 1 0"
-                origin_rpy="0 0 0" origin_xyz="0.025 0.0123 0.011"
+                origin_rpy="0 0 0" origin_xyz="0.025 ${coxa_thigh_dy} ${coxa_thigh_dz}"
                 parent="${link_10_name}" child="${link_11_name}" />
     <m_link_mesh name="${link_11_name}"
-                origin_rpy="1.57 0 3.14" origin_xyz="0.020 0.002 -0.007"
+                origin_rpy="${pi/2} 0 ${pi}" origin_xyz="${thigh_dx} 0.002 -${thigh_dy}"
                 mass="0.024357719"
                 ixx="0.0051411124" ixy="-0.00057530255" ixz="-0.000024729049"
@@ -190,5 +190,5 @@
                 parent="${link_11_name}" child="${link_12_name}" />
     <m_link_mesh name="${link_12_name}"
-                origin_rpy="4.712 0 0" origin_xyz="-0.008 -0.0197 0.023"
+                origin_rpy="${3*pi/2} 0 0" origin_xyz="-${tibia_dx} -${thigh_dz - tibia_dz} ${tibia_dy}"
                 mass="0.024357719"
                 ixx="0.0051411124" ixy="-0.00057530255" ixz="-0.000024729049"
@@ -202,8 +202,8 @@
                 type="revolute"
                 axis_xyz="0 0 1"
-                origin_rpy="0 0 0" origin_xyz="-0.040 0.078 -0.0112"
+                origin_rpy="0 0 0" origin_xyz="-${body_legs_dx} ${body_legs_r_dy} -${coxa_dz - body_legs_dz}"
                 parent="${link_00_name}" child="${link_13_name}" />
     <m_link_mesh name="${link_13_name}"
-                origin_rpy="3.14 0 0" origin_xyz="-0.033 -0.007 0"
+                origin_rpy="${pi} 0 0" origin_xyz="-${coxa_dx} -${coxa_dy} 0"
                 mass="0.024357719"
                 ixx="0.0051411124" ixy="-0.00057530255" ixz="-0.000024729049"
@@ -216,8 +216,8 @@
                 type="revolute"
                 axis_xyz="0 1 0"
-                origin_rpy="0 0 3.14" origin_xyz="-0.025 0.0123 0.011"
+                origin_rpy="0 0 ${pi}" origin_xyz="-0.025 ${coxa_thigh_dy} ${coxa_thigh_dz}"
                 parent="${link_13_name}" child="${link_14_name}" />
     <m_link_mesh name="${link_14_name}"
-                origin_rpy="1.57 0 0" origin_xyz="0.020 -0.002 -0.007"
+                origin_rpy="${pi/2} 0 0" origin_xyz="${thigh_dx} -0.002 -${thigh_dy}"
                 mass="0.024357719"
                 ixx="0.0051411124" ixy="-0.00057530255" ixz="-0.000024729049"
@@ -233,5 +233,5 @@
                 parent="${link_14_name}" child="${link_15_name}" />
     <m_link_mesh name="${link_15_name}"
-                origin_rpy="4.712 0 3.14" origin_xyz="-0.008 0.0197 0.023"
+                origin_rpy="${3*pi/2} 0 ${pi}" origin_xyz="-${tibia_dx} ${thigh_dz - tibia_dz} ${tibia_dy}"
                 mass="0.024357719"
                 ixx="0.0051411124" ixy="-0.00057530255" ixz="-0.000024729049"
@@ -245,8 +245,8 @@
                 type="revolute"
                 axis_xyz="0 0 1"
-                origin_rpy="0 0 0" origin_xyz="0.040 0.078 -0.0112"
+                origin_rpy="0 0 0" origin_xyz="${body_legs_dx} ${body_legs_r_dy} -${coxa_dz - body_legs_dz}"
                 parent="${link_00_name}" child="${link_16_name}" />
     <m_link_mesh name="${link_16_name}"
-                origin_rpy="3.14 0 0" origin_xyz="0.033 -0.007 0"
+                origin_rpy="${pi} 0 0" origin_xyz="${coxa_dx} -${coxa_dy} 0"
                 mass="0.024357719"
                 ixx="0.0051411124" ixy="-0.00057530255" ixz="-0.000024729049"
@@ -259,8 +259,8 @@
                 type="revolute"
                 axis_xyz="0 1 0"
-                origin_rpy="0 0 0" origin_xyz="0.025 0.0123 0.011"
+                origin_rpy="0 0 0" origin_xyz="0.025 ${coxa_thigh_dy} ${coxa_thigh_dz}"
                 parent="${link_16_name}" child="${link_17_name}" />
     <m_link_mesh name="${link_17_name}"
-                origin_rpy="1.57 0 3.14" origin_xyz="0.020 0.002 -0.007"
+                origin_rpy="${pi/2} 0 ${pi}" origin_xyz="${thigh_dx} 0.002 -${thigh_dy}"
                 mass="0.024357719"
                 ixx="0.0051411124" ixy="-0.00057530255" ixz="-0.000024729049"
@@ -276,5 +276,5 @@
                 parent="${link_17_name}" child="${link_18_name}" />
     <m_link_mesh name="${link_18_name}"
-                origin_rpy="4.712 0 0" origin_xyz="-0.008 -0.0197 0.023"
+                origin_rpy="${3*pi/2} 0 0" origin_xyz="-${tibia_dx} -${thigh_dz - tibia_dz} ${tibia_dy}"
                 mass="0.024357719"
                 ixx="0.0051411124" ixy="-0.00057530255" ixz="-0.000024729049"

File: urdf/robot_parameters.xacro (robot description, xacro)
@@ -20,3 +20,21 @@
     <xacro:property name="link_17_name" value="thigh_lr" />
     <xacro:property name="link_18_name" value="tibia_lr" />
+    <!-- Attachments params -->
+    <xacro:property name="body_legs_f_dy" value="0.066" />
+    <xacro:property name="body_legs_m_dy" value="0.006" />
+    <xacro:property name="body_legs_r_dy" value="0.078" />
+    <xacro:property name="body_legs_dx" value="0.04" />
+    <xacro:property name="body_legs_dz" value="0.0203" />
+    <xacro:property name="coxa_dx" value="0.033" />
+    <xacro:property name="coxa_dy" value="0.007" />
+    <xacro:property name="coxa_dz" value="0.0315" />
+    <xacro:property name="coxa_thigh_dx" value="0.008" />
+    <xacro:property name="coxa_thigh_dy" value="0.0123" />
+    <xacro:property name="coxa_thigh_dz" value="0.011" />
+    <xacro:property name="thigh_dx" value="0.02" />
+    <xacro:property name="thigh_dy" value="0.007" />
+    <xacro:property name="thigh_dz" value="0.032" />
+    <xacro:property name="tibia_dx" value="0.008" />
+    <xacro:property name="tibia_dy" value="0.023" />
+    <xacro:property name="tibia_dz" value="0.0123" />
 </robot>
