Commit message: Fix URDF, replace numbers on left leg

File: urdf/hexapod.xacro (robot description, xacro)
@@ -18,10 +18,11 @@
     </joint>
     <m_link_mesh name="body"
-                origin_rpy="0 0 0" origin_xyz="0 0 0"
+                origin_rpy="0 0 0"
+                origin_xyz="0 0 0"
                 mass="0.97559947"
                 ixx="3.1081800" ixy="-0.25460189" ixz="2.0318174"
                 iyy="6.3787776" iyz="0.16417863"
                 izz="5.3316425"
-                mesh_file="package://hexapod_description/meshes/body.stl"
+                mesh_file="package://hexapod_description/meshes/body"
                 mesh_scale="0.001 0.001 0.001" />
     <!-- Leg 1 (rf) begin description -->
@@ -30,13 +31,16 @@
                 type="revolute"
                 axis_xyz="0 0 1"
-                origin_rpy="0 0 0" origin_xyz="-${body_legs_dx} -${body_legs_f_dy} ${body_legs_dz}"
-                parent="body" child="${link_01_name}" />
+                origin_rpy="0 0 0"
+                origin_xyz="-${body_legs_dx} -${body_legs_f_dy} ${body_legs_dz}"
+                parent="body"
+                child="${link_01_name}" />
     <m_link_mesh name="${link_01_name}"
-                origin_rpy="${pi} 0 0" origin_xyz="-${coxa_dx} -${coxa_dy} -${coxa_dz}"
-                mass="0.024357719"
-                ixx="0.0051411124" ixy="-0.00057530255" ixz="-0.000024729049"
-                iyy="0.0081915737" iyz="-0.000019223094"
-                izz="0.0011379812"
-                mesh_file="package://hexapod_description/meshes/coxa_r.stl"
+                origin_rpy="${pi} 0 0"
+                origin_xyz="-${coxa_dx} -${coxa_dy} -${coxa_dz}"
+                mass="0.024357719"
+                ixx="0.0051411124" ixy="-0.00057530255" ixz="-0.000024729049"
+                iyy="0.0081915737" iyz="-0.000019223094"
+                izz="0.0011379812"
+                mesh_file="package://hexapod_description/meshes/coxa_r"
                 mesh_scale="0.001 0.001 0.001" />
     <!-- Leg 1 (rf) thigh description -->
@@ -44,13 +48,16 @@
                 type="revolute"
                 axis_xyz="0 1 0"
-                origin_rpy="0 0 ${pi}" origin_xyz="-${coxa_dx - coxa_thigh_dx} ${coxa_dy - coxa_thigh_dy} -${coxa_dz - coxa_thigh_dz}"
-                parent="${link_01_name}" child="${link_02_name}" />
+                origin_rpy="0 0 ${pi}"
+                origin_xyz="-${coxa_dx - coxa_thigh_dx} ${coxa_dy - coxa_thigh_dy} -${coxa_dz - coxa_thigh_dz}"
+                parent="${link_01_name}"
+                child="${link_02_name}" />
     <m_link_mesh name="${link_02_name}"
-                origin_rpy="${pi/2} 0 0" origin_xyz="${thigh_dx} -${thigh_dz - coxa_thigh_dy} -${thigh_dy}"
-                mass="0.024357719"
-                ixx="0.0051411124" ixy="-0.00057530255" ixz="-0.000024729049"
-                iyy="0.0081915737" iyz="-0.000019223094"
-                izz="0.0011379812"
-                mesh_file="package://hexapod_description/meshes/thigh.stl"
+                origin_rpy="${pi/2} 0 0"
+                origin_xyz="${thigh_dx} -${thigh_dz - coxa_thigh_dy} -${thigh_dy}"
+                mass="0.024357719"
+                ixx="0.0051411124" ixy="-0.00057530255" ixz="-0.000024729049"
+                iyy="0.0081915737" iyz="-0.000019223094"
+                izz="0.0011379812"
+                mesh_file="package://hexapod_description/meshes/thigh"
                 mesh_scale="0.001 0.001 0.001" />
     <!-- Leg 1 (rf) tibia description -->
@@ -58,13 +65,16 @@
                 type="revolute"
                 axis_xyz="0 1 0"
-                origin_rpy="0 0 0" origin_xyz="${thigh_dx * 2} -${thigh_dz - tibia_dz - 0.001} 0"
-                parent="${link_02_name}" child="${link_03_name}" />
+                origin_rpy="0 0 0"
+                origin_xyz="${thigh_dx * 2} -${thigh_dz - tibia_dz - 0.001} 0"
+                parent="${link_02_name}"
+                child="${link_03_name}" />
     <m_link_mesh name="${link_03_name}"
-                origin_rpy="${3*pi/2} 0 ${pi}" origin_xyz="-${tibia_dx} ${thigh_dz - tibia_dz} ${tibia_dy}"
-                mass="0.024357719"
-                ixx="0.0051411124" ixy="-0.00057530255" ixz="-0.000024729049"
-                iyy="0.0081915737" iyz="-0.000019223094"
-                izz="0.0011379812"
-                mesh_file="package://hexapod_description/meshes/tibia_r.stl"
+                origin_rpy="${3*pi/2} 0 ${pi}"
+                origin_xyz="-${tibia_dx} ${thigh_dz - tibia_dz} ${tibia_dy}"
+                mass="0.024357719"
+                ixx="0.0051411124" ixy="-0.00057530255" ixz="-0.000024729049"
+                iyy="0.0081915737" iyz="-0.000019223094"
+                izz="0.0011379812"
+                mesh_file="package://hexapod_description/meshes/tibia_r"
                 mesh_scale="0.001 0.001 0.001" />
     <!-- Leg 2 (lf) begin description -->
@@ -73,13 +83,16 @@
                 type="revolute"
                 axis_xyz="0 0 1"
-                origin_rpy="0 0 0" origin_xyz="${body_legs_dx} -${body_legs_f_dy} -${coxa_dz - body_legs_dz}"
-                parent="${link_00_name}" child="${link_04_name}" />
+                origin_rpy="0 0 0"
+                origin_xyz="${body_legs_dx} -${body_legs_f_dy} ${body_legs_dz}"
+                parent="${link_00_name}"
+                child="${link_04_name}" />
     <m_link_mesh name="${link_04_name}"
-                origin_rpy="${pi} 0 0" origin_xyz="${coxa_dx} -${coxa_dy} 0"
-                mass="0.024357719"
-                ixx="0.0051411124" ixy="-0.00057530255" ixz="-0.000024729049"
-                iyy="0.0081915737" iyz="-0.000019223094"
-                izz="0.0011379812"
-                mesh_file="package://hexapod_description/meshes/coxa_l.stl"
+                origin_rpy="${pi} 0 0"
+                origin_xyz="${coxa_dx} -${coxa_dy} -${coxa_dz}"
+                mass="0.024357719"
+                ixx="0.0051411124" ixy="-0.00057530255" ixz="-0.000024729049"
+                iyy="0.0081915737" iyz="-0.000019223094"
+                izz="0.0011379812"
+                mesh_file="package://hexapod_description/meshes/coxa_l"
                 mesh_scale="0.001 0.001 0.001" />
     <!-- Leg 2 (lf) thigh description -->
@@ -87,13 +100,16 @@
                 type="revolute"
                 axis_xyz="0 1 0"
-                origin_rpy="0 0 0" origin_xyz="0.025 ${coxa_thigh_dy} ${coxa_thigh_dz}"
-                parent="${link_04_name}" child="${link_05_name}" />
+                origin_rpy="0 0 0"
+                origin_xyz="${coxa_dx - coxa_thigh_dx} ${coxa_dy - coxa_thigh_dy} -${coxa_dz - coxa_thigh_dz}"
+                parent="${link_04_name}"
+                child="${link_05_name}" />
     <m_link_mesh name="${link_05_name}"
-                origin_rpy="${pi/2} 0 ${pi}" origin_xyz="${thigh_dx} 0.002 -${thigh_dy}"
-                mass="0.024357719"
-                ixx="0.0051411124" ixy="-0.00057530255" ixz="-0.000024729049"
-                iyy="0.0081915737" iyz="-0.000019223094"
-                izz="0.0011379812"
-                mesh_file="package://hexapod_description/meshes/thigh.stl"
+                origin_rpy="${pi/2} 0 ${pi}"
+                origin_xyz="${thigh_dx} ${thigh_dz - coxa_thigh_dy} -${thigh_dy}"
+                mass="0.024357719"
+                ixx="0.0051411124" ixy="-0.00057530255" ixz="-0.000024729049"
+                iyy="0.0081915737" iyz="-0.000019223094"
+                izz="0.0011379812"
+                mesh_file="package://hexapod_description/meshes/thigh"
                 mesh_scale="0.001 0.001 0.001" />
     <!-- Leg 2 (lf) tibia description -->
@@ -101,13 +117,16 @@
                 type="revolute"
                 axis_xyz="0 1 0"
-                origin_rpy="0 0 0" origin_xyz="0.040 0 0"
-                parent="${link_05_name}" child="${link_06_name}" />
+                origin_rpy="0 0 0"
+                origin_xyz="${thigh_dx * 2} ${thigh_dz - tibia_dz - 0.001} 0"
+                parent="${link_05_name}"
+                child="${link_06_name}" />
     <m_link_mesh name="${link_06_name}"
-                origin_rpy="${3*pi/2} 0 0" origin_xyz="-${tibia_dx} -${thigh_dz - tibia_dz} ${tibia_dy}"
-                mass="0.024357719"
-                ixx="0.0051411124" ixy="-0.00057530255" ixz="-0.000024729049"
-                iyy="0.0081915737" iyz="-0.000019223094"
-                izz="0.0011379812"
-                mesh_file="package://hexapod_description/meshes/tibia_l.stl"
+                origin_rpy="${3*pi/2} 0 0"
+                origin_xyz="-${tibia_dx} -${thigh_dz - tibia_dz} ${tibia_dy}"
+                mass="0.024357719"
+                ixx="0.0051411124" ixy="-0.00057530255" ixz="-0.000024729049"
+                iyy="0.0081915737" iyz="-0.000019223094"
+                izz="0.0011379812"
+                mesh_file="package://hexapod_description/meshes/tibia_l"
                 mesh_scale="0.001 0.001 0.001" />
     <!-- Leg 3 (rm) begin description -->
@@ -116,13 +135,16 @@
                 type="revolute"
                 axis_xyz="0 0 1"
-                origin_rpy="0 0 0" origin_xyz="-${body_legs_dx} ${body_legs_m_dy} -${coxa_dz - body_legs_dz}"
-                parent="${link_00_name}" child="${link_07_name}" />
+                origin_rpy="0 0 0"
+                origin_xyz="-${body_legs_dx} ${body_legs_m_dy} -${coxa_dz - body_legs_dz}"
+                parent="${link_00_name}"
+                child="${link_07_name}" />
     <m_link_mesh name="${link_07_name}"
-                origin_rpy="${pi} 0 0" origin_xyz="-${coxa_dx} -${coxa_dy} 0"
-                mass="0.024357719"
-                ixx="0.0051411124" ixy="-0.00057530255" ixz="-0.000024729049"
-                iyy="0.0081915737" iyz="-0.000019223094"
-                izz="0.0011379812"
-                mesh_file="package://hexapod_description/meshes/coxa_r.stl"
+                origin_rpy="${pi} 0 0"
+                origin_xyz="-${coxa_dx} -${coxa_dy} 0"
+                mass="0.024357719"
+                ixx="0.0051411124" ixy="-0.00057530255" ixz="-0.000024729049"
+                iyy="0.0081915737" iyz="-0.000019223094"
+                izz="0.0011379812"
+                mesh_file="package://hexapod_description/meshes/coxa_r"
                 mesh_scale="0.001 0.001 0.001" />
     <!-- Leg 3 (rm) thigh description -->
@@ -130,13 +152,16 @@
                 type="revolute"
                 axis_xyz="0 1 0"
-                origin_rpy="0 0 ${pi}" origin_xyz="-0.025 ${coxa_thigh_dy} ${coxa_thigh_dz}"
-                parent="${link_07_name}" child="${link_08_name}" />
+                origin_rpy="0 0 ${pi}"
+                origin_xyz="-0.025 ${coxa_thigh_dy} ${coxa_thigh_dz}"
+                parent="${link_07_name}"
+                child="${link_08_name}" />
     <m_link_mesh name="${link_08_name}"
-                origin_rpy="${pi/2} 0 0" origin_xyz="${thigh_dx} -0.002 -${thigh_dy}"
-                mass="0.024357719"
-                ixx="0.0051411124" ixy="-0.00057530255" ixz="-0.000024729049"
-                iyy="0.0081915737" iyz="-0.000019223094"
-                izz="0.0011379812"
-                mesh_file="package://hexapod_description/meshes/thigh.stl"
+                origin_rpy="${pi/2} 0 0"
+                origin_xyz="${thigh_dx} -0.002 -${thigh_dy}"
+                mass="0.024357719"
+                ixx="0.0051411124" ixy="-0.00057530255" ixz="-0.000024729049"
+                iyy="0.0081915737" iyz="-0.000019223094"
+                izz="0.0011379812"
+                mesh_file="package://hexapod_description/meshes/thigh"
                 mesh_scale="0.001 0.001 0.001" />
     <!-- Leg 3 (rm) tibia description -->
@@ -144,13 +169,16 @@
                 type="revolute"
                 axis_xyz="0 1 0"
-                origin_rpy="0 0 0" origin_xyz="0.040 0 0"
-                parent="${link_08_name}" child="${link_09_name}" />
+                origin_rpy="0 0 0"
+                origin_xyz="0.040 0 0"
+                parent="${link_08_name}"
+                child="${link_09_name}" />
     <m_link_mesh name="${link_09_name}"
-                origin_rpy="${3*pi/2} 0 ${pi}" origin_xyz="-${tibia_dx} ${thigh_dz - tibia_dz} ${tibia_dy}"
-                mass="0.024357719"
-                ixx="0.0051411124" ixy="-0.00057530255" ixz="-0.000024729049"
-                iyy="0.0081915737" iyz="-0.000019223094"
-                izz="0.0011379812"
-                mesh_file="package://hexapod_description/meshes/tibia_r.stl"
+                origin_rpy="${3*pi/2} 0 ${pi}"
+                origin_xyz="-${tibia_dx} ${thigh_dz - tibia_dz} ${tibia_dy}"
+                mass="0.024357719"
+                ixx="0.0051411124" ixy="-0.00057530255" ixz="-0.000024729049"
+                iyy="0.0081915737" iyz="-0.000019223094"
+                izz="0.0011379812"
+                mesh_file="package://hexapod_description/meshes/tibia_r"
                 mesh_scale="0.001 0.001 0.001" />
     <!-- Leg 4 (lm) begin description -->
@@ -159,13 +187,16 @@
                 type="revolute"
                 axis_xyz="0 0 1"
-                origin_rpy="0 0 0" origin_xyz="${body_legs_dx} ${body_legs_m_dy} -${coxa_dz - body_legs_dz}"
-                parent="${link_00_name}" child="${link_10_name}" />
+                origin_rpy="0 0 0"
+                origin_xyz="${body_legs_dx} ${body_legs_m_dy} -${coxa_dz - body_legs_dz}"
+                parent="${link_00_name}"
+                child="${link_10_name}" />
     <m_link_mesh name="${link_10_name}"
-                origin_rpy="${pi} 0 0" origin_xyz="${coxa_dx} -${coxa_dy} 0"
-                mass="0.024357719"
-                ixx="0.0051411124" ixy="-0.00057530255" ixz="-0.000024729049"
-                iyy="0.0081915737" iyz="-0.000019223094"
-                izz="0.0011379812"
-                mesh_file="package://hexapod_description/meshes/coxa_l.stl"
+                origin_rpy="${pi} 0 0"
+                origin_xyz="${coxa_dx} -${coxa_dy} 0"
+                mass="0.024357719"
+                ixx="0.0051411124" ixy="-0.00057530255" ixz="-0.000024729049"
+                iyy="0.0081915737" iyz="-0.000019223094"
+                izz="0.0011379812"
+                mesh_file="package://hexapod_description/meshes/coxa_l"
                 mesh_scale="0.001 0.001 0.001" />
     <!-- Leg 4 (lm) thigh description -->
@@ -173,13 +204,16 @@
                 type="revolute"
                 axis_xyz="0 1 0"
-                origin_rpy="0 0 0" origin_xyz="0.025 ${coxa_thigh_dy} ${coxa_thigh_dz}"
-                parent="${link_10_name}" child="${link_11_name}" />
+                origin_rpy="0 0 0"
+                origin_xyz="0.025 ${coxa_thigh_dy} ${coxa_thigh_dz}"
+                parent="${link_10_name}"
+                child="${link_11_name}" />
     <m_link_mesh name="${link_11_name}"
-                origin_rpy="${pi/2} 0 ${pi}" origin_xyz="${thigh_dx} 0.002 -${thigh_dy}"
-                mass="0.024357719"
-                ixx="0.0051411124" ixy="-0.00057530255" ixz="-0.000024729049"
-                iyy="0.0081915737" iyz="-0.000019223094"
-                izz="0.0011379812"
-                mesh_file="package://hexapod_description/meshes/thigh.stl"
+                origin_rpy="${pi/2} 0 ${pi}"
+                origin_xyz="${thigh_dx} 0.002 -${thigh_dy}"
+                mass="0.024357719"
+                ixx="0.0051411124" ixy="-0.00057530255" ixz="-0.000024729049"
+                iyy="0.0081915737" iyz="-0.000019223094"
+                izz="0.0011379812"
+                mesh_file="package://hexapod_description/meshes/thigh"
                 mesh_scale="0.001 0.001 0.001" />
     <!-- Leg 4 (lm) tibia description -->
@@ -187,13 +221,16 @@
                 type="revolute"
                 axis_xyz="0 1 0"
-                origin_rpy="0 0 0" origin_xyz="0.040 0 0"
-                parent="${link_11_name}" child="${link_12_name}" />
+                origin_rpy="0 0 0"
+                origin_xyz="0.040 0 0"
+                parent="${link_11_name}"
+                child="${link_12_name}" />
     <m_link_mesh name="${link_12_name}"
-                origin_rpy="${3*pi/2} 0 0" origin_xyz="-${tibia_dx} -${thigh_dz - tibia_dz} ${tibia_dy}"
-                mass="0.024357719"
-                ixx="0.0051411124" ixy="-0.00057530255" ixz="-0.000024729049"
-                iyy="0.0081915737" iyz="-0.000019223094"
-                izz="0.0011379812"
-                mesh_file="package://hexapod_description/meshes/tibia_l.stl"
+                origin_rpy="${3*pi/2} 0 0"
+                origin_xyz="-${tibia_dx} -${thigh_dz - tibia_dz} ${tibia_dy}"
+                mass="0.024357719"
+                ixx="0.0051411124" ixy="-0.00057530255" ixz="-0.000024729049"
+                iyy="0.0081915737" iyz="-0.000019223094"
+                izz="0.0011379812"
+                mesh_file="package://hexapod_description/meshes/tibia_l"
                 mesh_scale="0.001 0.001 0.001" />
     <!-- Leg 5 (rr) begin description -->
@@ -202,13 +239,16 @@
                 type="revolute"
                 axis_xyz="0 0 1"
-                origin_rpy="0 0 0" origin_xyz="-${body_legs_dx} ${body_legs_r_dy} -${coxa_dz - body_legs_dz}"
-                parent="${link_00_name}" child="${link_13_name}" />
+                origin_rpy="0 0 0"
+                origin_xyz="-${body_legs_dx} ${body_legs_r_dy} -${coxa_dz - body_legs_dz}"
+                parent="${link_00_name}"
+                child="${link_13_name}" />
     <m_link_mesh name="${link_13_name}"
-                origin_rpy="${pi} 0 0" origin_xyz="-${coxa_dx} -${coxa_dy} 0"
-                mass="0.024357719"
-                ixx="0.0051411124" ixy="-0.00057530255" ixz="-0.000024729049"
-                iyy="0.0081915737" iyz="-0.000019223094"
-                izz="0.0011379812"
-                mesh_file="package://hexapod_description/meshes/coxa_r.stl"
+                origin_rpy="${pi} 0 0"
+                origin_xyz="-${coxa_dx} -${coxa_dy} 0"
+                mass="0.024357719"
+                ixx="0.0051411124" ixy="-0.00057530255" ixz="-0.000024729049"
+                iyy="0.0081915737" iyz="-0.000019223094"
+                izz="0.0011379812"
+                mesh_file="package://hexapod_description/meshes/coxa_r"
                 mesh_scale="0.001 0.001 0.001" />
     <!-- Leg 5 (rr) thigh description -->
@@ -216,13 +256,16 @@
                 type="revolute"
                 axis_xyz="0 1 0"
-                origin_rpy="0 0 ${pi}" origin_xyz="-0.025 ${coxa_thigh_dy} ${coxa_thigh_dz}"
-                parent="${link_13_name}" child="${link_14_name}" />
+                origin_rpy="0 0 ${pi}"
+                origin_xyz="-0.025 ${coxa_thigh_dy} ${coxa_thigh_dz}"
+                parent="${link_13_name}"
+                child="${link_14_name}" />
     <m_link_mesh name="${link_14_name}"
-                origin_rpy="${pi/2} 0 0" origin_xyz="${thigh_dx} -0.002 -${thigh_dy}"
-                mass="0.024357719"
-                ixx="0.0051411124" ixy="-0.00057530255" ixz="-0.000024729049"
-                iyy="0.0081915737" iyz="-0.000019223094"
-                izz="0.0011379812"
-                mesh_file="package://hexapod_description/meshes/thigh.stl"
+                origin_rpy="${pi/2} 0 0"
+                origin_xyz="${thigh_dx} -0.002 -${thigh_dy}"
+                mass="0.024357719"
+                ixx="0.0051411124" ixy="-0.00057530255" ixz="-0.000024729049"
+                iyy="0.0081915737" iyz="-0.000019223094"
+                izz="0.0011379812"
+                mesh_file="package://hexapod_description/meshes/thigh"
                 mesh_scale="0.001 0.001 0.001" />
     <!-- Leg 5 (rr) tibia description -->
@@ -230,13 +273,16 @@
                 type="revolute"
                 axis_xyz="0 1 0"
-                origin_rpy="0 0 0" origin_xyz="0.040 0 0"
-                parent="${link_14_name}" child="${link_15_name}" />
+                origin_rpy="0 0 0"
+                origin_xyz="0.040 0 0"
+                parent="${link_14_name}"
+                child="${link_15_name}" />
     <m_link_mesh name="${link_15_name}"
-                origin_rpy="${3*pi/2} 0 ${pi}" origin_xyz="-${tibia_dx} ${thigh_dz - tibia_dz} ${tibia_dy}"
-                mass="0.024357719"
-                ixx="0.0051411124" ixy="-0.00057530255" ixz="-0.000024729049"
-                iyy="0.0081915737" iyz="-0.000019223094"
-                izz="0.0011379812"
-                mesh_file="package://hexapod_description/meshes/tibia_r.stl"
+                origin_rpy="${3*pi/2} 0 ${pi}"
+                origin_xyz="-${tibia_dx} ${thigh_dz - tibia_dz} ${tibia_dy}"
+                mass="0.024357719"
+                ixx="0.0051411124" ixy="-0.00057530255" ixz="-0.000024729049"
+                iyy="0.0081915737" iyz="-0.000019223094"
+                izz="0.0011379812"
+                mesh_file="package://hexapod_description/meshes/tibia_r"
                 mesh_scale="0.001 0.001 0.001" />
     <!-- Leg 6 (lr) begin description -->
@@ -245,13 +291,16 @@
                 type="revolute"
                 axis_xyz="0 0 1"
-                origin_rpy="0 0 0" origin_xyz="${body_legs_dx} ${body_legs_r_dy} -${coxa_dz - body_legs_dz}"
-                parent="${link_00_name}" child="${link_16_name}" />
+                origin_rpy="0 0 0"
+                origin_xyz="${body_legs_dx} ${body_legs_r_dy} -${coxa_dz - body_legs_dz}"
+                parent="${link_00_name}"
+                child="${link_16_name}" />
     <m_link_mesh name="${link_16_name}"
-                origin_rpy="${pi} 0 0" origin_xyz="${coxa_dx} -${coxa_dy} 0"
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
File: urdf/links_joints.xacro (robot description, xacro)
@@ -31,5 +31,5 @@
                 <origin rpy="${origin_rpy}" xyz="${origin_xyz}" />
                 <geometry>
-                    <mesh filename="${mesh_file}" scale="${mesh_scale}" />
+                    <mesh filename="${mesh_file}_coll.stl" scale="${mesh_scale}" />
                 </geometry>
             </collision>
@@ -37,5 +37,5 @@
                 <origin rpy="${origin_rpy}" xyz="${origin_xyz}" />
                 <geometry>
-                    <mesh filename="${mesh_file}" scale="${mesh_scale}" />
+                    <mesh filename="${mesh_file}.stl" scale="${mesh_scale}" />
                 </geometry>
                 <material name="light_black" />
