Commit message: Add legs macro

File: urdf/hexapod.xacro (robot description, xacro)
@@ -3,4 +3,5 @@
     <xacro:include filename="$(find hexapod_description)/urdf/links_joints.xacro" />
     <xacro:include filename="$(find hexapod_description)/urdf/robot_parameters.xacro" />
+    <xacro:include filename="$(find hexapod_description)/urdf/legs.xacro" />
     <xacro:include filename="$(find hexapod_description)/urdf/camera.xacro" />
     <link name="base_link"/>
@@ -26,316 +27,40 @@
                 mesh_file="package://hexapod_description/meshes/body"
                 mesh_scale="0.001 0.001 0.001" />
-    <!-- Leg 1 (rf) begin description -->
-    <!-- Leg 1 (rf) coxa description -->
-    <m_joint    name="${link_01_name}"
-                type="revolute"
-                axis_xyz="0 0 1"
-                origin_rpy="0 0 0"
-                origin_xyz="-${body_legs_dx} -${body_legs_f_dy} ${body_legs_dz}"
-                parent="body"
-                child="${link_01_name}" />
-    <m_link_mesh name="${link_01_name}"
-                origin_rpy="${pi} 0 0"
-                origin_xyz="-${coxa_dx} -${coxa_dy} -${coxa_dz}"
-                mass="0.024357719"
-                ixx="0.0051411124" ixy="-0.00057530255" ixz="-0.000024729049"
-                iyy="0.0081915737" iyz="-0.000019223094"
-                izz="0.0011379812"
-                mesh_file="package://hexapod_description/meshes/coxa_r"
-                mesh_scale="0.001 0.001 0.001" />
-    <!-- Leg 1 (rf) thigh description -->
-    <m_joint    name="${link_02_name}"
-                type="revolute"
-                axis_xyz="0 1 0"
-                origin_rpy="0 0 ${pi}"
-                origin_xyz="-${coxa_dx - coxa_thigh_dx} ${coxa_dy - coxa_thigh_dy} -${coxa_dz - coxa_thigh_dz}"
-                parent="${link_01_name}"
-                child="${link_02_name}" />
-    <m_link_mesh name="${link_02_name}"
-                origin_rpy="${pi/2} 0 0"
-                origin_xyz="${thigh_dx} -${thigh_dz - coxa_thigh_dy} -${thigh_dy}"
-                mass="0.024357719"
-                ixx="0.0051411124" ixy="-0.00057530255" ixz="-0.000024729049"
-                iyy="0.0081915737" iyz="-0.000019223094"
-                izz="0.0011379812"
-                mesh_file="package://hexapod_description/meshes/thigh"
-                mesh_scale="0.001 0.001 0.001" />
-    <!-- Leg 1 (rf) tibia description -->
-    <m_joint    name="${link_03_name}"
-                type="revolute"
-                axis_xyz="0 1 0"
-                origin_rpy="0 0 0"
-                origin_xyz="${thigh_dx * 2} -${thigh_dz - tibia_dz - 0.001} 0"
-                parent="${link_02_name}"
-                child="${link_03_name}" />
-    <m_link_mesh name="${link_03_name}"
-                origin_rpy="${3*pi/2} 0 ${pi}"
-                origin_xyz="-${tibia_dx} ${thigh_dz - tibia_dz} ${tibia_dy}"
-                mass="0.024357719"
-                ixx="0.0051411124" ixy="-0.00057530255" ixz="-0.000024729049"
-                iyy="0.0081915737" iyz="-0.000019223094"
-                izz="0.0011379812"
-                mesh_file="package://hexapod_description/meshes/tibia_r"
-                mesh_scale="0.001 0.001 0.001" />
-    <!-- Leg 2 (lf) begin description -->
-    <!-- Leg 2 (lf) coxa description -->
-    <m_joint    name="${link_04_name}"
-                type="revolute"
-                axis_xyz="0 0 1"
-                origin_rpy="0 0 0"
-                origin_xyz="${body_legs_dx} -${body_legs_f_dy} ${body_legs_dz}"
-                parent="${link_00_name}"
-                child="${link_04_name}" />
-    <m_link_mesh name="${link_04_name}"
-                origin_rpy="${pi} 0 0"
-                origin_xyz="${coxa_dx} -${coxa_dy} -${coxa_dz}"
-                mass="0.024357719"
-                ixx="0.0051411124" ixy="-0.00057530255" ixz="-0.000024729049"
-                iyy="0.0081915737" iyz="-0.000019223094"
-                izz="0.0011379812"
-                mesh_file="package://hexapod_description/meshes/coxa_l"
-                mesh_scale="0.001 0.001 0.001" />
-    <!-- Leg 2 (lf) thigh description -->
-    <m_joint    name="${link_05_name}"
-                type="revolute"
-                axis_xyz="0 1 0"
-                origin_rpy="0 0 0"
-                origin_xyz="${coxa_dx - coxa_thigh_dx} ${coxa_dy - coxa_thigh_dy} -${coxa_dz - coxa_thigh_dz}"
-                parent="${link_04_name}"
-                child="${link_05_name}" />
-    <m_link_mesh name="${link_05_name}"
-                origin_rpy="${pi/2} 0 ${pi}"
-                origin_xyz="${thigh_dx} ${thigh_dz - coxa_thigh_dy} -${thigh_dy}"
-                mass="0.024357719"
-                ixx="0.0051411124" ixy="-0.00057530255" ixz="-0.000024729049"
-                iyy="0.0081915737" iyz="-0.000019223094"
-                izz="0.0011379812"
-                mesh_file="package://hexapod_description/meshes/thigh"
-                mesh_scale="0.001 0.001 0.001" />
-    <!-- Leg 2 (lf) tibia description -->
-    <m_joint    name="${link_06_name}"
-                type="revolute"
-                axis_xyz="0 1 0"
-                origin_rpy="0 0 0"
-                origin_xyz="${thigh_dx * 2} ${thigh_dz - tibia_dz - 0.001} 0"
-                parent="${link_05_name}"
-                child="${link_06_name}" />
-    <m_link_mesh name="${link_06_name}"
-                origin_rpy="${3*pi/2} 0 0"
-                origin_xyz="-${tibia_dx} -${thigh_dz - tibia_dz} ${tibia_dy}"
-                mass="0.024357719"
-                ixx="0.0051411124" ixy="-0.00057530255" ixz="-0.000024729049"
-                iyy="0.0081915737" iyz="-0.000019223094"
-                izz="0.0011379812"
-                mesh_file="package://hexapod_description/meshes/tibia_l"
-                mesh_scale="0.001 0.001 0.001" />
-    <!-- Leg 3 (rm) begin description -->
-    <!-- Leg 3 (rm) coxa description -->
-    <m_joint    name="${link_07_name}"
-                type="revolute"
-                axis_xyz="0 0 1"
-                origin_rpy="0 0 0"
-                origin_xyz="-${body_legs_dx} ${body_legs_m_dy} -${coxa_dz - body_legs_dz}"
-                parent="${link_00_name}"
-                child="${link_07_name}" />
-    <m_link_mesh name="${link_07_name}"
-                origin_rpy="${pi} 0 0"
-                origin_xyz="-${coxa_dx} -${coxa_dy} 0"
-                mass="0.024357719"
-                ixx="0.0051411124" ixy="-0.00057530255" ixz="-0.000024729049"
-                iyy="0.0081915737" iyz="-0.000019223094"
-                izz="0.0011379812"
-                mesh_file="package://hexapod_description/meshes/coxa_r"
-                mesh_scale="0.001 0.001 0.001" />
-    <!-- Leg 3 (rm) thigh description -->
-    <m_joint    name="${link_08_name}"
-                type="revolute"
-                axis_xyz="0 1 0"
-                origin_rpy="0 0 ${pi}"
-                origin_xyz="-0.025 ${coxa_thigh_dy} ${coxa_thigh_dz}"
-                parent="${link_07_name}"
-                child="${link_08_name}" />
-    <m_link_mesh name="${link_08_name}"
-                origin_rpy="${pi/2} 0 0"
-                origin_xyz="${thigh_dx} -0.002 -${thigh_dy}"
-                mass="0.024357719"
-                ixx="0.0051411124" ixy="-0.00057530255" ixz="-0.000024729049"
-                iyy="0.0081915737" iyz="-0.000019223094"
-                izz="0.0011379812"
-                mesh_file="package://hexapod_description/meshes/thigh"
-                mesh_scale="0.001 0.001 0.001" />
-    <!-- Leg 3 (rm) tibia description -->
-    <m_joint    name="${link_09_name}"
-                type="revolute"
-                axis_xyz="0 1 0"
-                origin_rpy="0 0 0"
-                origin_xyz="0.040 0 0"
-                parent="${link_08_name}"
-                child="${link_09_name}" />
-    <m_link_mesh name="${link_09_name}"
-                origin_rpy="${3*pi/2} 0 ${pi}"
-                origin_xyz="-${tibia_dx} ${thigh_dz - tibia_dz} ${tibia_dy}"
-                mass="0.024357719"
-                ixx="0.0051411124" ixy="-0.00057530255" ixz="-0.000024729049"
-                iyy="0.0081915737" iyz="-0.000019223094"
-                izz="0.0011379812"
-                mesh_file="package://hexapod_description/meshes/tibia_r"
-                mesh_scale="0.001 0.001 0.001" />
-    <!-- Leg 4 (lm) begin description -->
-    <!-- Leg 4 (lm) coxa description -->
-    <m_joint    name="${link_10_name}"
-                type="revolute"
-                axis_xyz="0 0 1"
-                origin_rpy="0 0 0"
-                origin_xyz="${body_legs_dx} ${body_legs_m_dy} -${coxa_dz - body_legs_dz}"
-                parent="${link_00_name}"
-                child="${link_10_name}" />
-    <m_link_mesh name="${link_10_name}"
-                origin_rpy="${pi} 0 0"
-                origin_xyz="${coxa_dx} -${coxa_dy} 0"
-                mass="0.024357719"
-                ixx="0.0051411124" ixy="-0.00057530255" ixz="-0.000024729049"
-                iyy="0.0081915737" iyz="-0.000019223094"
-                izz="0.0011379812"
-                mesh_file="package://hexapod_description/meshes/coxa_l"
-                mesh_scale="0.001 0.001 0.001" />
-    <!-- Leg 4 (lm) thigh description -->
-    <m_joint    name="${link_11_name}"
-                type="revolute"
-                axis_xyz="0 1 0"
-                origin_rpy="0 0 0"
-                origin_xyz="0.025 ${coxa_thigh_dy} ${coxa_thigh_dz}"
-                parent="${link_10_name}"
-                child="${link_11_name}" />
-    <m_link_mesh name="${link_11_name}"
-                origin_rpy="${pi/2} 0 ${pi}"
-                origin_xyz="${thigh_dx} 0.002 -${thigh_dy}"
-                mass="0.024357719"
-                ixx="0.0051411124" ixy="-0.00057530255" ixz="-0.000024729049"
-                iyy="0.0081915737" iyz="-0.000019223094"
-                izz="0.0011379812"
-                mesh_file="package://hexapod_description/meshes/thigh"
-                mesh_scale="0.001 0.001 0.001" />
-    <!-- Leg 4 (lm) tibia description -->
-    <m_joint    name="${link_12_name}"
-                type="revolute"
-                axis_xyz="0 1 0"
-                origin_rpy="0 0 0"
-                origin_xyz="0.040 0 0"
-                parent="${link_11_name}"
-                child="${link_12_name}" />
-    <m_link_mesh name="${link_12_name}"
-                origin_rpy="${3*pi/2} 0 0"
-                origin_xyz="-${tibia_dx} -${thigh_dz - tibia_dz} ${tibia_dy}"
-                mass="0.024357719"
-                ixx="0.0051411124" ixy="-0.00057530255" ixz="-0.000024729049"
-                iyy="0.0081915737" iyz="-0.000019223094"
-                izz="0.0011379812"
-                mesh_file="package://hexapod_description/meshes/tibia_l"
-                mesh_scale="0.001 0.001 0.001" />
-    <!-- Leg 5 (rr) begin description -->
-    <!-- Leg 5 (rr) coxa description -->
-    <m_joint    name="${link_13_name}"
-                type="revolute"
-                axis_xyz="0 0 1"
-                origin_rpy="0 0 0"
-                origin_xyz="-${body_legs_dx} ${body_legs_r_dy} -${coxa_dz - body_legs_dz}"
-                parent="${link_00_name}"
-                child="${link_13_name}" />
-    <m_link_mesh name="${link_13_name}"
-                origin_rpy="${pi} 0 0"
-                origin_xyz="-${coxa_dx} -${coxa_dy} 0"
-                mass="0.024357719"
-                ixx="0.0051411124" ixy="-0.00057530255" ixz="-0.000024729049"
-                iyy="0.0081915737" iyz="-0.000019223094"
-                izz="0.0011379812"
-                mesh_file="package://hexapod_description/meshes/coxa_r"
-                mesh_scale="0.001 0.001 0.001" />
-    <!-- Leg 5 (rr) thigh description -->
-    <m_joint    name="${link_14_name}"
-                type="revolute"
-                axis_xyz="0 1 0"
-                origin_rpy="0 0 ${pi}"
-                origin_xyz="-0.025 ${coxa_thigh_dy} ${coxa_thigh_dz}"
-                parent="${link_13_name}"
-                child="${link_14_name}" />
-    <m_link_mesh name="${link_14_name}"
-                origin_rpy="${pi/2} 0 0"
-                origin_xyz="${thigh_dx} -0.002 -${thigh_dy}"
-                mass="0.024357719"
-                ixx="0.0051411124" ixy="-0.00057530255" ixz="-0.000024729049"
-                iyy="0.0081915737" iyz="-0.000019223094"
-                izz="0.0011379812"
-                mesh_file="package://hexapod_description/meshes/thigh"
-                mesh_scale="0.001 0.001 0.001" />
-    <!-- Leg 5 (rr) tibia description -->
-    <m_joint    name="${link_15_name}"
-                type="revolute"
-                axis_xyz="0 1 0"
-                origin_rpy="0 0 0"
-                origin_xyz="0.040 0 0"
-                parent="${link_14_name}"
-                child="${link_15_name}" />
-    <m_link_mesh name="${link_15_name}"
-                origin_rpy="${3*pi/2} 0 ${pi}"
-                origin_xyz="-${tibia_dx} ${thigh_dz - tibia_dz} ${tibia_dy}"
-                mass="0.024357719"
-                ixx="0.0051411124" ixy="-0.00057530255" ixz="-0.000024729049"
-                iyy="0.0081915737" iyz="-0.000019223094"
-                izz="0.0011379812"
-                mesh_file="package://hexapod_description/meshes/tibia_r"
-                mesh_scale="0.001 0.001 0.001" />
-    <!-- Leg 6 (lr) begin description -->
-    <!-- Leg 6 (lr) coxa description -->
-    <m_joint    name="${link_16_name}"
-                type="revolute"
-                axis_xyz="0 0 1"
-                origin_rpy="0 0 0"
-                origin_xyz="${body_legs_dx} ${body_legs_r_dy} -${coxa_dz - body_legs_dz}"
-                parent="${link_00_name}"
-                child="${link_16_name}" />
-    <m_link_mesh name="${link_16_name}"
-                origin_rpy="${pi} 0 0"
-                origin_xyz="${coxa_dx} -${coxa_dy} 0"
-                mass="0.024357719"
-                ixx="0.0051411124" ixy="-0.00057530255" ixz="-0.000024729049"
-                iyy="0.0081915737" iyz="-0.000019223094"
-                izz="0.0011379812"
-                mesh_file="package://hexapod_description/meshes/coxa_l"
-                mesh_scale="0.001 0.001 0.001" />
-    <!-- Leg 6 (lr) thigh description -->
-    <m_joint    name="${link_17_name}"
-                type="revolute"
-                axis_xyz="0 1 0"
-                origin_rpy="0 0 0"
-                origin_xyz="0.025 ${coxa_thigh_dy} ${coxa_thigh_dz}"
-                parent="${link_16_name}"
-                child="${link_17_name}" />
-    <m_link_mesh name="${link_17_name}"
-                origin_rpy="${pi/2} 0 ${pi}"
-                origin_xyz="${thigh_dx} 0.002 -${thigh_dy}"
-                mass="0.024357719"
-                ixx="0.0051411124" ixy="-0.00057530255" ixz="-0.000024729049"
-                iyy="0.0081915737" iyz="-0.000019223094"
-                izz="0.0011379812"
-                mesh_file="package://hexapod_description/meshes/thigh"
-                mesh_scale="0.001 0.001 0.001" />
-    <!-- Leg 6 (lr) tibia description -->
-    <m_joint    name="${link_18_name}"
-                type="revolute"
-                axis_xyz="0 1 0"
-                origin_rpy="0 0 0"
-                origin_xyz="0.040 0 0"
-                parent="${link_17_name}"
-                child="${link_18_name}" />
-    <m_link_mesh name="${link_18_name}"
-                origin_rpy="${3*pi/2} 0 0"
-                origin_xyz="-${tibia_dx} -${thigh_dz - tibia_dz} ${tibia_dy}"
-                mass="0.024357719"
-                ixx="0.0051411124" ixy="-0.00057530255" ixz="-0.000024729049"
-                iyy="0.0081915737" iyz="-0.000019223094"
-                izz="0.0011379812"
-                mesh_file="package://hexapod_description/meshes/tibia_l"
-                mesh_scale="0.001 0.001 0.001" />
+    <!-- Leg 1 (rf) description -->
+    <m_leg_r    body_leg_dy="${body_legs_f_dy}"
+                body_link_name="${link_00_name}"
+                coxa_link_name="${link_01_name}"
+                thigh_link_name="${link_02_name}"
+                tibia_link_name="${link_03_name}" />
+    <!-- Leg 2 (lf) description -->
+    <m_leg_l    body_leg_dy="${body_legs_f_dy}"
+                body_link_name="${link_00_name}"
+                coxa_link_name="${link_04_name}"
+                thigh_link_name="${link_05_name}"
+                tibia_link_name="${link_06_name}" />
+    <!-- Leg 3 (rm) description -->
+    <m_leg_r    body_leg_dy="${body_legs_m_dy}"
+                body_link_name="${link_00_name}"
+                coxa_link_name="${link_07_name}"
+                thigh_link_name="${link_08_name}"
+                tibia_link_name="${link_09_name}" />
+    <!-- Leg 4 (lm) description -->
+    <m_leg_l    body_leg_dy="${body_legs_m_dy}"
+                body_link_name="${link_00_name}"
+                coxa_link_name="${link_10_name}"
+                thigh_link_name="${link_11_name}"
+                tibia_link_name="${link_12_name}" />
+    <!-- Leg 5 (rr) description -->
+    <m_leg_r    body_leg_dy="${body_legs_r_dy}"
+                body_link_name="${link_00_name}"
+                coxa_link_name="${link_13_name}"
+                thigh_link_name="${link_14_name}"
+                tibia_link_name="${link_15_name}" />
+    <!-- Leg 6 (lr) description -->
+    <m_leg_l    body_leg_dy="${body_legs_r_dy}"
+                body_link_name="${link_00_name}"
+                coxa_link_name="${link_16_name}"
+                thigh_link_name="${link_17_name}"
+                tibia_link_name="${link_18_name}" />
     <gazebo>
         <plugin name="gazebo_ros_control" filename="libgazebo_ros_control.so">

File: urdf/robot_parameters.xacro (robot description, xacro)
@@ -21,5 +21,5 @@
     <xacro:property name="link_18_name" value="tibia_lr" />
     <!-- Attachments params -->
-    <xacro:property name="body_legs_f_dy" value="0.066" />
+    <xacro:property name="body_legs_f_dy" value="-0.066" />
     <xacro:property name="body_legs_m_dy" value="0.006" />
     <xacro:property name="body_legs_r_dy" value="0.078" />
