Commit message: Fixed description, updated control, added rc.

File: hexapod_description/urdf/hexapod.xacro (robot description, xacro)
@@ -9,5 +9,5 @@
         <parent link="base_link"/>
         <child link="body"/>
-        <origin rpy="0 0 ${pi/2}" xyz="0 0 0"/>
+        <origin rpy="0 0 0" xyz="0 0 0"/>
     </joint>
     <xacro:my_camera/>
@@ -18,15 +18,16 @@
       <child link="camera_link"/>
     </joint>
-    <m_link_mesh name="body"
+    <simple_mesh_link name="body"
                 origin_rpy="0 0 0"
                 origin_xyz="0 0 0"
-                mass="0.97559947"
-                ixx="3.1081800" ixy="-0.25460189" ixz="2.0318174"
-                iyy="6.3787776" iyz="0.16417863"
-                izz="5.3316425"
+                com_xyz="${body_com_x} ${body_com_y} ${body_com_z}"
+                mass="0.1"
+                ixx="${0.140413 / i_div}" ixy="${0 / i_div}" ixz="${0.000026 / i_div}"
+                iyy="${0.378107 / i_div}" iyz="${0 / i_div}"
+                izz=" ${0.512999 /i_div}"
                 mesh_file="package://hexapod_description/meshes/body"
                 mesh_scale="0.001 0.001 0.001" />
     <!-- Leg 1 (rf) description -->
-    <m_leg_r    body_leg_dy="${body_legs_f_dy}"
+    <leg_r    body_leg_dx="${body_legs_f_dx}"
                 body_link_name="${link_00_name}"
                 coxa_link_name="${link_01_name}"
@@ -34,5 +35,5 @@
                 tibia_link_name="${link_03_name}" />
     <!-- Leg 2 (lf) description -->
-    <m_leg_l    body_leg_dy="${body_legs_f_dy}"
+    <leg_l    body_leg_dx="${body_legs_f_dx}"
                 body_link_name="${link_00_name}"
                 coxa_link_name="${link_04_name}"
@@ -40,5 +41,5 @@
                 tibia_link_name="${link_06_name}" />
     <!-- Leg 3 (rm) description -->
-    <m_leg_r    body_leg_dy="${body_legs_m_dy}"
+    <leg_r    body_leg_dx="${body_legs_m_dx}"
                 body_link_name="${link_00_name}"
                 coxa_link_name="${link_07_name}"
@@ -46,5 +47,5 @@
                 tibia_link_name="${link_09_name}" />
     <!-- Leg 4 (lm) description -->
-    <m_leg_l    body_leg_dy="${body_legs_m_dy}"
+    <leg_l    body_leg_dx="${body_legs_m_dx}"
                 body_link_name="${link_00_name}"
                 coxa_link_name="${link_10_name}"
@@ -52,5 +53,5 @@
                 tibia_link_name="${link_12_name}" />
     <!-- Leg 5 (rr) description -->
-    <m_leg_r    body_leg_dy="${body_legs_r_dy}"
+    <leg_r    body_leg_dx="${body_legs_r_dx}"
                 body_link_name="${link_00_name}"
                 coxa_link_name="${link_13_name}"
@@ -58,5 +59,5 @@
                 tibia_link_name="${link_15_name}" />
     <!-- Leg 6 (lr) description -->
-    <m_leg_l    body_leg_dy="${body_legs_r_dy}"
+    <leg_l    body_leg_dx="${body_legs_r_dx}"
                 body_link_name="${link_00_name}"
                 coxa_link_name="${link_16_name}"

File: hexapod_description/urdf/legs.xacro (robot description, xacro)
@@ -3,110 +3,116 @@
     <xacro:include filename="$(find hexapod_description)/urdf/robot_parameters.xacro" />
     <xacro:include filename="$(find hexapod_description)/urdf/links_joints.xacro" />
-    <xacro:macro    name = "m_leg_l"
-                    params = "body_leg_dy body_link_name coxa_link_name thigh_link_name tibia_link_name" >
+    <xacro:macro    name = "leg_l"
+                    params = "body_leg_dx body_link_name coxa_link_name thigh_link_name tibia_link_name" >
         <!-- Coxa description -->
-        <m_joint    name="${coxa_link_name}"
+        <simple_joint name="${coxa_link_name}"
                     type="revolute"
                     axis_xyz="0 0 1"
                     origin_rpy="0 0 0"
-                    origin_xyz="${body_legs_dx} ${body_leg_dy} ${body_legs_dz}"
+                    origin_xyz="${body_leg_dx} ${body_legs_dy} ${body_legs_dz}"
                     parent="${body_link_name}"
                     child="${coxa_link_name}" />
-        <m_link_mesh name="${coxa_link_name}"
-                    origin_rpy="${pi} 0 0"
-                    origin_xyz="${coxa_dx} -${coxa_dy} -${coxa_dz}"
-                    mass="0.024357719"
-                    ixx="0.0051411124" ixy="-0.00057530255" ixz="-0.000024729049"
-                    iyy="0.0081915737" iyz="-0.000019223094"
-                    izz="0.0011379812"
+        <simple_mesh_link name="${coxa_link_name}"
+                    origin_rpy="0 0 0"
+                    origin_xyz="${coxa_dx} ${coxa_dy} ${coxa_dz}"
+                    com_xyz="${coxa_com_x + coxa_dx} ${-coxa_com_y + coxa_dy} ${coxa_com_z + coxa_dz}"
+                    mass="0.011"
+                    ixx="0.001827" ixy="-0.000062" ixz="0.000016"
+                    iyy="0.001496" iyz="0.000151"
+                    izz="0.001137"
                     mesh_file="package://hexapod_description/meshes/coxa_l"
                     mesh_scale="0.001 0.001 0.001" />
         <!-- Thigh description -->
-        <m_joint    name="${thigh_link_name}"
+        <simple_joint    name="${thigh_link_name}"
                     type="revolute"
-                    axis_xyz="0 1 0"
-                    origin_rpy="0 0 0"
-                    origin_xyz="${coxa_dx - coxa_thigh_dx} ${coxa_dy - coxa_thigh_dy} -${coxa_dz - coxa_thigh_dz}"
+                    axis_xyz="1 0 0"
+                    origin_rpy="0 ${pi} 0"
+                    origin_xyz="${coxa_dx + coxa_thigh_dx} ${coxa_dy - coxa_thigh_dy} ${coxa_dz - coxa_thigh_dz}"
                     parent="${coxa_link_name}"
                     child="${thigh_link_name}" />
-        <m_link_mesh name="${thigh_link_name}"
-                    origin_rpy="${pi/2} 0 ${pi}"
-                    origin_xyz="${thigh_dx} ${thigh_dz - coxa_thigh_dy} -${thigh_dy}"
-                    mass="0.024357719"
-                    ixx="0.0051411124" ixy="-0.00057530255" ixz="-0.000024729049"
-                    iyy="0.0081915737" iyz="-0.000019223094"
-                    izz="0.0011379812"
+        <simple_mesh_link name="${thigh_link_name}"
+                    origin_rpy="0 ${pi} 0"
+                    origin_xyz="${thigh_dx} ${thigh_dy} ${thigh_dz}"
+                    com_xyz="${-thigh_com_x + thigh_dx} ${thigh_com_y + thigh_dy} ${thigh_com_z}"
+                    mass="0.004"
+                    ixx="0.000844" ixy="0" ixz="-0.000015"
+                    iyy="0.000959" iyz="0"
+                    izz="0.001661"
                     mesh_file="package://hexapod_description/meshes/thigh"
                     mesh_scale="0.001 0.001 0.001" />
         <!-- Leg 2 (lf) tibia description -->
-        <m_joint    name="${tibia_link_name}"
+        <simple_joint    name="${tibia_link_name}"
                     type="revolute"
-                    axis_xyz="0 1 0"
+                    axis_xyz="1 0 0"
                     origin_rpy="0 0 0"
-                    origin_xyz="${thigh_dx * 2} ${thigh_dz - tibia_dz - 0.001} 0"
+                    origin_xyz="0 ${thigh_dy * 2} 0"
                     parent="${thigh_link_name}"
                     child="${tibia_link_name}" />
-        <m_link_mesh name="${tibia_link_name}"
-                    origin_rpy="${3*pi/2} 0 0"
-                    origin_xyz="-${tibia_dx} -${thigh_dz - tibia_dz} ${tibia_dy}"
-                    mass="0.024357719"
-                    ixx="0.0051411124" ixy="-0.00057530255" ixz="-0.000024729049"
-                    iyy="0.0081915737" iyz="-0.000019223094"
-                    izz="0.0011379812"
-                    mesh_file="package://hexapod_description/meshes/tibia_l"
+        <simple_mesh_link name="${tibia_link_name}"
+                    origin_rpy="0 ${pi} 0"
+                    origin_xyz="${tibia_dx} ${-tibia_dy} ${-tibia_dz}"
+                    com_xyz="${-tibia_com_x + tibia_dx} ${tibia_com_y - tibia_dy} ${tibia_com_z + tibia_dz}"
+                    mass="0.011"
+                    ixx="0.003738" ixy="0" ixz="-0.000029"
+                    iyy="0.003919" iyz="0"
+                    izz="0.00059"
+                    mesh_file="package://hexapod_description/meshes/tibia"
                     mesh_scale="0.001 0.001 0.001" />
     </xacro:macro>
-    <xacro:macro    name = "m_leg_r"
-                    params = "body_leg_dy body_link_name coxa_link_name thigh_link_name tibia_link_name" >
+    <xacro:macro    name = "leg_r"
+                    params = "body_leg_dx body_link_name coxa_link_name thigh_link_name tibia_link_name" >
         <!-- Coxa description -->
-        <m_joint    name="${coxa_link_name}"
+        <simple_joint    name="${coxa_link_name}"
                     type="revolute"
                     axis_xyz="0 0 1"
                     origin_rpy="0 0 0"
-                    origin_xyz="-${body_legs_dx} ${body_leg_dy} ${body_legs_dz}"
+                    origin_xyz="${body_leg_dx} -${body_legs_dy} ${body_legs_dz}"
                     parent="${body_link_name}"
                     child="${coxa_link_name}" />
-        <m_link_mesh name="${coxa_link_name}"
-                    origin_rpy="${pi} 0 0"
-                    origin_xyz="-${coxa_dx} -${coxa_dy} -${coxa_dz}"
-                    mass="0.024357719"
-                    ixx="0.0051411124" ixy="-0.00057530255" ixz="-0.000024729049"
-                    iyy="0.0081915737" iyz="-0.000019223094"
-                    izz="0.0011379812"
+        <simple_mesh_link name="${coxa_link_name}"
+                    origin_rpy="0 0 0"
+                    origin_xyz="${coxa_dx} -${coxa_dy} ${coxa_dz}"
+                    com_xyz="${coxa_com_x + coxa_dx} ${coxa_com_y - coxa_dy} ${coxa_com_z + coxa_dz}"
+                    mass="0.011"
+                    ixx="0.001827" ixy="0.000062" ixz="0.000016"
+                    iyy="0.001496" iyz="-0.000151"
+                    izz="0.001137"
                     mesh_file="package://hexapod_description/meshes/coxa_r"
                     mesh_scale="0.001 0.001 0.001" />
         <!-- Thigh description -->
-        <m_joint    name="${thigh_link_name}"
+        <simple_joint    name="${thigh_link_name}"
                     type="revolute"
-                    axis_xyz="0 1 0"
-                    origin_rpy="0 0 ${pi}"
-                    origin_xyz="-${coxa_dx - coxa_thigh_dx} ${coxa_dy - coxa_thigh_dy} -${coxa_dz - coxa_thigh_dz}"
+                    axis_xyz="1 0 0"
+                    origin_rpy="0 0 0"
+                    origin_xyz="${coxa_dx + coxa_thigh_dx} ${-coxa_dy + coxa_thigh_dy} ${coxa_dz - coxa_thigh_dz}"
                     parent="${coxa_link_name}"
                     child="${thigh_link_name}" />
-        <m_link_mesh name="${thigh_link_name}"
-                    origin_rpy="${pi/2} 0 0"
-                    origin_xyz="${thigh_dx} -${thigh_dz - coxa_thigh_dy} -${thigh_dy}"
-                    mass="0.024357719"
-                    ixx="0.0051411124" ixy="-0.00057530255" ixz="-0.000024729049"
-                    iyy="0.0081915737" iyz="-0.000019223094"
-                    izz="0.0011379812"
+        <simple_mesh_link name="${thigh_link_name}"
+                    origin_rpy="0 0 0"
+                    origin_xyz="${-thigh_dx} ${-thigh_dy} ${-thigh_dz}"
+                    com_xyz="${thigh_com_x - thigh_dx} ${thigh_com_y - thigh_dy} ${thigh_com_z}"
+                    mass="0.004"
+                    ixx="0.000844" ixy="0" ixz="-0.000015"
+                    iyy="0.000959" iyz="0"
+                    izz="0.001661"
                     mesh_file="package://hexapod_description/meshes/thigh"
                     mesh_scale="0.001 0.001 0.001" />
         <!-- Tibia description -->
-        <m_joint    name="${tibia_link_name}"
+        <simple_joint    name="${tibia_link_name}"
                     type="revolute"
-                    axis_xyz="0 1 0"
+                    axis_xyz="1 0 0"
                     origin_rpy="0 0 0"
-                    origin_xyz="${thigh_dx * 2} -${thigh_dz - tibia_dz - 0.001} 0"
+                    origin_xyz="0 ${-thigh_dy * 2} 0"
                     parent="${thigh_link_name}"
                     child="${tibia_link_name}" />
-        <m_link_mesh name="${tibia_link_name}"
-                    origin_rpy="${3*pi/2} 0 ${pi}"
-                    origin_xyz="-${tibia_dx} ${thigh_dz - tibia_dz} ${tibia_dy}"
-                    mass="0.024357719"
-                    ixx="0.0051411124" ixy="-0.00057530255" ixz="-0.000024729049"
-                    iyy="0.0081915737" iyz="-0.000019223094"
-                    izz="0.0011379812"
-                    mesh_file="package://hexapod_description/meshes/tibia_r"
+        <simple_mesh_link name="${tibia_link_name}"
+                    origin_rpy="0 0 0"
+                    origin_xyz="${-tibia_dx} ${tibia_dy} ${tibia_dz}"
+                    com_xyz="${tibia_com_x - tibia_dx} ${tibia_com_y - tibia_dy} ${tibia_com_z + tibia_dz}"
+                    mass="0.011"
+                    ixx="0.003738" ixy="0" ixz="-0.000029"
+                    iyy="0.003919" iyz="0"
+                    izz="0.00059"
+                    mesh_file="package://hexapod_description/meshes/tibia"
                     mesh_scale="0.001 0.001 0.001" />
     </xacro:macro>

File: hexapod_description/urdf/links_joints.xacro (robot description, xacro)
@@ -1,9 +1,8 @@
 <?xml version="1.0" ?>
 <robot xmlns:xacro="http://www.ros.org/wiki/xacro">
-    <xacro:macro name="m_joint" params="name type axis_xyz origin_rpy origin_xyz parent child">
+    <xacro:macro name="simple_joint" params="name type axis_xyz origin_rpy origin_xyz parent child">
         <joint name="j_${name}" type="${type}">
             <axis xyz="${axis_xyz}" />
-            <!--<limit effort="${limit_e}" lower="${limit_l}" upper="${limit_u}" velocity="${limit_v}" />-->
-            <limit effort="2.8" lower="-2.6179939" upper="2.6179939" velocity="5.6548668"/>
+            <limit effort="15" lower="-${pi/2}" upper="${pi/2}" velocity="5"/>
             <origin rpy="${origin_rpy}" xyz="${origin_xyz}" />
             <parent link="${parent}" />
@@ -21,9 +20,11 @@
         </transmission>
     </xacro:macro>
-    <xacro:macro name="m_link_mesh" params="name origin_rpy origin_xyz mesh_file mesh_scale mass ixx ixy ixz iyy iyz izz">
+    <xacro:macro
+        name="simple_mesh_link"
+        params="name origin_rpy origin_xyz com_xyz mesh_file mesh_scale mass ixx ixy ixz iyy iyz izz">
         <link name="${name}">
             <inertial>
                 <mass value="${mass}" />
-                <origin rpy="${origin_rpy}" xyz="${origin_xyz}" />
+                <origin rpy="${origin_rpy}" xyz="${com_xyz}" />
                 <inertia ixx="${ixx}" ixy="${ixy}" ixz="${ixz}" iyy="${iyy}" iyz="${iyz}" izz="${izz}" />
             </inertial>
@@ -33,12 +34,4 @@
                     <mesh filename="${mesh_file}_coll.stl" scale="${mesh_scale}" />
                 </geometry>
-                <surface>
-                    <friction>
-                        <ode>
-                            <mu>1</mu>
-                            <mu2>1</mu2>
-                        </ode>
-                    </friction>
-                </surface>
             </collision>
             <visual>
@@ -51,47 +44,3 @@
         </link>
     </xacro:macro>
-    <!--
-    <xacro:macro name="m_link_cylinder" params="name origin_rpy origin_xyz radius length mass ixx ixy ixz iyy iyz izz">
-        <link name="${name}">
-            <inertial>
-                <mass value="${mass}" />
-                <origin rpy="${origin_rpy}" xyz="${origin_xyz}" />
-                <inertia ixx="${ixx}" ixy="${ixy}" ixz="${ixz}" iyy="${iyy}" iyz="${iyz}" izz="${izz}" />
-            </inertial>
-            <collision>
-                <origin rpy="${origin_rpy}" xyz="${origin_xyz}" />
-                <geometry>
-                    <cylinder radius="${radius}" length="${length}" />
-                </geometry>
-            </collision>
-            <visual>
-                <origin rpy="${origin_rpy}" xyz="${origin_xyz}" />
-                <geometry>
-                    <cylinder radius="${radius}" length="${length}" />
-                </geometry>
-            </visual>
-        </link>
-    </xacro:macro>
-    <xacro:macro name="m_link_box" params="name origin_rpy origin_xyz size mass ixx ixy ixz iyy iyz izz">
-        <link name="${name}">
-            <inertial>
-                <mass value="${mass}" />
-                <origin rpy="${origin_rpy}" xyz="${origin_xyz}" />
-                <inertia ixx="${ixx}" ixy="${ixy}" ixz="${ixz}" iyy="${iyy}" iyz="${iyz}" izz="${izz}" />
-            </inertial>
-            <collision>
-                <origin rpy="${origin_rpy}" xyz="${origin_xyz}" />
-                <geometry>
-                    <box size="${size}" />
-                </geometry>
-            </collision>
-            <visual>
-                <origin rpy="${origin_rpy}" xyz="${origin_xyz}" />
-                <geometry>
-                    <box size="${size}" />
-                </geometry>
-            </visual>
-        </link>
-    </xacro:macro>
-    -->
 </robot>

File: hexapod_description/urdf/robot_parameters.xacro (robot description, xacro)
@@ -1,40 +1,62 @@
 <?xml version="1.0" ?>
 <robot xmlns:xacro="http://www.ros.org/wiki/xacro">
+    <!-- Links list -->
     <xacro:property name="link_00_name" value="body" />
-    <xacro:property name="link_01_name" value="c1_rf" />
+    <xacro:property name="link_01_name" value="coxa_rf" />
     <xacro:property name="link_02_name" value="thigh_rf" />
     <xacro:property name="link_03_name" value="tibia_rf" />
-    <xacro:property name="link_04_name" value="c1_lf" />
+    <xacro:property name="link_04_name" value="coxa_lf" />
     <xacro:property name="link_05_name" value="thigh_lf" />
     <xacro:property name="link_06_name" value="tibia_lf" />
-    <xacro:property name="link_07_name" value="c1_rm" />
+    <xacro:property name="link_07_name" value="coxa_rm" />
     <xacro:property name="link_08_name" value="thigh_rm" />
     <xacro:property name="link_09_name" value="tibia_rm" />
-    <xacro:property name="link_10_name" value="c1_lm" />
+    <xacro:property name="link_10_name" value="coxa_lm" />
     <xacro:property name="link_11_name" value="thigh_lm" />
     <xacro:property name="link_12_name" value="tibia_lm" />
-    <xacro:property name="link_13_name" value="c1_rr" />
+    <xacro:property name="link_13_name" value="coxa_rr" />
     <xacro:property name="link_14_name" value="thigh_rr" />
     <xacro:property name="link_15_name" value="tibia_rr" />
-    <xacro:property name="link_16_name" value="c1_lr" />
+    <xacro:property name="link_16_name" value="coxa_lr" />
     <xacro:property name="link_17_name" value="thigh_lr" />
     <xacro:property name="link_18_name" value="tibia_lr" />
-    <!-- Attachments params -->
-    <xacro:property name="body_legs_f_dy" value="-0.066" />
-    <xacro:property name="body_legs_m_dy" value="0.006" />
-    <xacro:property name="body_legs_r_dy" value="0.078" />
-    <xacro:property name="body_legs_dx" value="0.04" />
-    <xacro:property name="body_legs_dz" value="0.0203" />
-    <xacro:property name="coxa_dx" value="0.033" />
-    <xacro:property name="coxa_dy" value="0.007" />
-    <xacro:property name="coxa_dz" value="0.0315" />
-    <xacro:property name="coxa_thigh_dx" value="0.008" />
-    <xacro:property name="coxa_thigh_dy" value="0.0123" />
-    <xacro:property name="coxa_thigh_dz" value="0.011" />
-    <xacro:property name="thigh_dx" value="0.02" />
-    <xacro:property name="thigh_dy" value="0.007" />
-    <xacro:property name="thigh_dz" value="0.032" />
-    <xacro:property name="tibia_dx" value="0.008" />
-    <xacro:property name="tibia_dy" value="0.023" />
-    <xacro:property name="tibia_dz" value="0.0123" />
+    <!-- Inertia params-->
+    <xacro:property name="i_div" value="1000.0"/>
+    <!-- Body params -->
+    <xacro:property name="body_legs_f_dx" value="0.066" />
+    <xacro:property name="body_legs_m_dx" value="-0.006" />
+    <xacro:property name="body_legs_r_dx" value="-0.078" />
+    <xacro:property name="body_legs_dy" value="0.04" />
+    <xacro:property name="body_legs_dz" value="0.0243" />
+    <!-- Center of Mass position-->
+    <xacro:property name="body_com_x" value="-0.000465" />
+    <xacro:property name="body_com_y" value="0" />
+    <xacro:property name="body_com_z" value="0.006191" />
+    <!-- Coxa params -->
+    <xacro:property name="coxa_dx" value="0.007" />
+    <xacro:property name="coxa_dy" value="0.033" />
+    <xacro:property name="coxa_dz" value="0.0025" />
+    <xacro:property name="coxa_thigh_dx" value="0.0123" />
+    <xacro:property name="coxa_thigh_dy" value="0.008" />
+    <xacro:property name="coxa_thigh_dz" value="0.023" />
+    <!-- Center of Mass position-->
+    <xacro:property name="coxa_com_x" value="-0.005038" />
+    <xacro:property name="coxa_com_y" value="0.010896" />
+    <xacro:property name="coxa_com_z" value="-0.01694" />
+    <!-- Thigh params -->
+    <xacro:property name="thigh_dx" value="0.01525" />
+    <xacro:property name="thigh_dy" value="0.02" />
+    <xacro:property name="thigh_dz" value="0" />
+    <!-- Center of Mass position-->
+    <xacro:property name="thigh_com_x" value="0.00504" />
+    <xacro:property name="thigh_com_y" value="0" />
+    <xacro:property name="thigh_com_z" value="-0.000293" />
+    <!-- Tibia params -->
+    <xacro:property name="tibia_dx" value="0.0123" />
+    <xacro:property name="tibia_dy" value="0" />
+    <xacro:property name="tibia_dz" value="0.023" />
+    <!-- Center of Mass position-->
+    <xacro:property name="tibia_com_x" value="-0.00471" />
+    <xacro:property name="tibia_com_y" value="0" />
+    <xacro:property name="tibia_com_z" value="-0.025056" />
 </robot>
